File: epaper-102.kicad_pcb (KiCad board)
At the start: 2 copper layers, 19.6 x 38.6 mm, 20 parts, among them J1 Conn_01x30_Female, J2 Conn_01x08_Female

Commit message: Add M2 mouting holes to pcb.
Parts:
- added REF**: MountingHole_2.2mm_M2_ISO7380_Pad_TopBottom, MountingHole:MountingHole_2.2mm_M2_ISO7380_Pad_TopBottom, F.Cu at (44.4, 95.8)
- added REF**: MountingHole_2.2mm_M2_ISO7380_Pad_TopBottom, MountingHole:MountingHole_2.2mm_M2_ISO7380_Pad_TopBottom, F.Cu at (22.3, 95.8)
Other:
- board size 19.6 x 38.6 mm -> 25.8 x 38.6 mm
- net class Default removed
